File: HardWare/BOM/Scope_F07x.kicad_pcb (KiCad board)
At the start: 2 copper layers, 38 x 37.8 mm, 131 parts, among them P1 CONN_X12, Q1 2N7002KW, SW1 Button-2P+PAD, SW2 Button-2P+PAD, SW3 Button-2P+PAD, SW4 Button-2P+PAD, SW5 Button-2P+PAD, U1 OPA4197, U2 STM32F072CBU6, U3 SGM8632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

Commit message: R4从750R修改为536R，原因是DAC输出缓冲器不是轨到轨，通过减小R4增加增益解决
Parts:
- R4: value 750R -> 536R

Commit message: RT9393更正为RT9193，添加3d打印模型
Parts:
- U2: value STM32F072CBU6 -> STM32F072CBU6 / STM32F071CBU6
- U4: value RT9393-33GB -> RT9193-33GB
